File: PCB/watch/watch.kicad_sch (KiCad schematic)
At the start: 1 part, among them U1 STM8S105S6T6C

Commit message: feat(pcb): Buncha stuff happened
Parts:
- removed U1: STM8S105S6T6C, LQFP-44, symbol STM8S105S6T6C:STM8S105S6T6C
- added U1: STM8S105C6T6, LQFP48-7X7mm, symbol STM8S105C6T6:STM8S105C6T6
Connections:
- new net +3V0: U1.5 (VSS)
